Commit message: Rebase from 'release/indigo/ur_description'

File: urdf/ur.transmission.xacro (robot description, xacro)
@@ -1,9 +1,9 @@
 <?xml version="1.0"?>
 <robot xmlns:xacro="http://www.ros.org/wiki/xacro">
-  <xacro:macro name="ur5_arm_transmission" params="prefix">
+  <xacro:macro name="ur_arm_transmission" params="prefix">
     <transmission name="${prefix}shoulder_pan_trans">
       <type>transmission_interface/SimpleTransmission</type>
       <joint name="${prefix}shoulder_pan_joint">
-        <hardwareInterface>EffortJointInterface</hardwareInterface>
+        <hardwareInterface>PositionJointInterface</hardwareInterface>
       </joint>
       <actuator name="${prefix}shoulder_pan_motor">
@@ -14,5 +14,5 @@
       <type>transmission_interface/SimpleTransmission</type>
       <joint name="${prefix}shoulder_lift_joint">
-        <hardwareInterface>EffortJointInterface</hardwareInterface>
+        <hardwareInterface>PositionJointInterface</hardwareInterface>
       </joint>
       <actuator name="${prefix}shoulder_lift_motor">
@@ -23,5 +23,5 @@
       <type>transmission_interface/SimpleTransmission</type>
       <joint name="${prefix}elbow_joint">
-        <hardwareInterface>EffortJointInterface</hardwareInterface>
+        <hardwareInterface>PositionJointInterface</hardwareInterface>
       </joint>
       <actuator name="${prefix}elbow_motor">
@@ -32,5 +32,5 @@
       <type>transmission_interface/SimpleTransmission</type>
       <joint name="${prefix}wrist_1_joint">
-        <hardwareInterface>EffortJointInterface</hardwareInterface>
+        <hardwareInterface>PositionJointInterface</hardwareInterface>
       </joint>
       <actuator name="${prefix}wrist_1_motor">
@@ -41,5 +41,5 @@
       <type>transmission_interface/SimpleTransmission</type>
       <joint name="${prefix}wrist_2_joint">
-        <hardwareInterface>EffortJointInterface</hardwareInterface>
+        <hardwareInterface>PositionJointInterface</hardwareInterface>
       </joint>
       <actuator name="${prefix}wrist_2_motor">
@@ -50,5 +50,5 @@
       <type>transmission_interface/SimpleTransmission</type>
       <joint name="${prefix}wrist_3_joint">
-        <hardwareInterface>EffortJointInterface</hardwareInterface>
+        <hardwareInterface>PositionJointInterface</hardwareInterface>
       </joint>
       <actuator name="${prefix}wrist_3_motor">

File: urdf/ur3.urdf.xacro (robot description, xacro)
@@ -2,6 +2,5 @@
 <robot xmlns:xacro="http://www.ros.org/wiki/xacro">
 <!--
-  Author: Kelsey Hawkins
-  Contributers: Jimmy Da Silva, Ajit Krisshna N L, Muhammad Asif Rana
+  Author: Felix Messmer
 -->
   <xacro:include filename="$(find ur_description)/urdf/ur.transmission.xacro" />
@@ -9,39 +8,39 @@
   <property name="pi" value="3.14159265" />
   <!-- Inertia parameters -->
-  <property name="base_mass" value="4.0" />  <!-- This mass might be incorrect -->
-  <property name="shoulder_mass" value="7.778" />
-  <property name="upper_arm_mass" value="12.93" />
-  <property name="forearm_mass" value="3.87" />
-  <property name="wrist_1_mass" value="1.96" />
-  <property name="wrist_2_mass" value="1.96" />
-  <property name="wrist_3_mass" value="0.202" />
+  <property name="base_mass" value="2.0" />  <!-- This mass might be incorrect -->
+  <property name="shoulder_mass" value="2.0" />
+  <property name="upper_arm_mass" value="3.42" />
+  <property name="forearm_mass" value="1.26" />
+  <property name="wrist_1_mass" value="0.8" />
+  <property name="wrist_2_mass" value="0.8" />
+  <property name="wrist_3_mass" value="0.35" />
   <!-- These parameters are borrowed from the urcontrol.conf file
        but are not verified for the correct permutation.
        The permutation was guessed by looking at the UR5 parameters.
        Serious use of these parameters needs further inspection. -->
-  <property name="shoulder_cog" value="0.00008 0.00244 -0.037" />
-  <property name="upper_arm_cog" value="0.00001 0.15061 0.38757" />
-  <property name="forearm_cog" value="-0.00012 0.06112 0.1984" />
-  <property name="wrist_1_cog" value="-0.00021 -0.00112 0.02269" />
-  <property name="wrist_2_cog" value="-0.00021 0.00112 0.002269" />
-  <property name="wrist_3_cog" value="0 -0.001156 -0.00149" />
+  <property name="shoulder_cog" value="0.0 -0.02 0.0" />
+  <property name="upper_arm_cog" value="0.13 0.0 0.1157" />
+  <property name="forearm_cog" value="0.05 0.0 0.0238" />
+  <property name="wrist_1_cog" value="0.0 0.0 0.01" />
+  <property name="wrist_2_cog" value="0.0 0.0 0.01" />
+  <property name="wrist_3_cog" value="0.0 0.0 -0.02" />
   <!-- Kinematic model -->
   <!-- Properties from urcontrol.conf -->
-  <property name="ur10_d1" value="0.1273" />
-  <property name="ur10_a2" value="-0.612" />
-  <property name="ur10_a3" value="-0.5723" />
-  <property name="ur10_d4" value="0.163941" />
-  <property name="ur10_d5" value="0.1157" />
-  <property name="ur10_d6" value="0.0922" />
+  <property name="ur3_d1" value="0.1519" />
+  <property name="ur3_a2" value="-0.24365" />
+  <property name="ur3_a3" value="-0.21325" />
+  <property name="ur3_d4" value="0.11235" />
+  <property name="ur3_d5" value="0.08535" />
+  <property name="ur3_d6" value="0.0819" />
   <!-- Arbitrary offsets for shoulder/elbow joints -->
-  <property name="shoulder_offset" value="0.220941" />  <!-- measured from model -->
-  <property name="elbow_offset" value="-0.1719" /> <!-- measured from model -->
+  <property name="shoulder_offset" value="0.1198" />  <!-- measured from model -->
+  <property name="elbow_offset" value="-0.0925" /> <!-- measured from model -->
   <!-- link lengths used in model -->
-  <property name="shoulder_height" value="${ur10_d1}" />
-  <property name="upper_arm_length" value="${-ur10_a2}" />
-  <property name="forearm_length" value="${-ur10_a3}" />
-  <property name="wrist_1_length" value="${ur10_d4 - elbow_offset - shoulder_offset}" />
-  <property name="wrist_2_length" value="${ur10_d5}" />
-  <property name="wrist_3_length" value="${ur10_d6}" />
+  <property name="shoulder_height" value="${ur3_d1}" />
+  <property name="upper_arm_length" value="${-ur3_a2}" />
+  <property name="forearm_length" value="${-ur3_a3}" />
+  <property name="wrist_1_length" value="${ur3_d4 - elbow_offset - shoulder_offset}" />
+  <property name="wrist_2_length" value="${ur3_d5}" />
+  <property name="wrist_3_length" value="${ur3_d6}" />
   <xacro:macro name="cylinder_inertial" params="radius length mass *origin">
     <inertial>
@@ -53,17 +52,17 @@
     </inertial>
   </xacro:macro>
-  <xacro:macro name="ur10_robot" params="prefix joint_limited">
+  <xacro:macro name="ur3_robot" params="prefix joint_limited">
     <link name="${prefix}base_link" >
       <visual>
         <geometry>
-          <mesh filename="package://ur_description/meshes/ur10/visual/base.dae"/>
-        </geometry>
-        <material name="LightGrey">
-          <color rgba="0.7 0.7 0.7 1.0"/>
-        </material>
-      </visual>
-      <collision>
-        <geometry>
-          <mesh filename="package://ur_description/meshes/ur10/collision/base.stl"/>
+          <mesh filename="package://ur_description/meshes/ur3/visual/base.dae"/>
+        </geometry>
+        <material name="LightGrey">
+          <color rgba="0.7 0.7 0.7 1.0"/>
+        </material>
+      </visual>
+      <collision>
+        <geometry>
+          <mesh filename="package://ur_description/meshes/ur3/collision/base.stl"/>
         </geometry>
       </collision>
@@ -88,13 +87,13 @@
       <visual>
         <geometry>
-          <mesh filename="package://ur_description/meshes/ur10/visual/shoulder.dae"/>
-        </geometry>
-        <material name="LightGrey">
-          <color rgba="0.7 0.7 0.7 1.0"/>
-        </material>
-      </visual>
-      <collision>
-        <geometry>
-          <mesh filename="package://ur_description/meshes/ur10/collision/shoulder.stl"/>
+          <mesh filename="package://ur_description/meshes/ur3/visual/shoulder.dae"/>
+        </geometry>
+        <material name="LightGrey">
+          <color rgba="0.7 0.7 0.7 1.0"/>
+        </material>
+      </visual>
+      <collision>
+        <geometry>
+          <mesh filename="package://ur_description/meshes/ur3/collision/shoulder.stl"/>
         </geometry>
       </collision>
@@ -119,17 +118,17 @@
       <visual>
         <geometry>
-          <mesh filename="package://ur_description/meshes/ur10/visual/upperarm.dae"/>
-        </geometry>
-        <material name="LightGrey">
-          <color rgba="0.7 0.7 0.7 1.0"/>
-        </material>
-      </visual>
-      <collision>
-        <geometry>
-          <mesh filename="package://ur_description/meshes/ur10/collision/upperarm.stl"/>
-        </geometry>
-      </collision>
-      <xacro:cylinder_inertial radius="0.075" length="${-ur10_a2}" mass="${upper_arm_mass}">
-        <origin xyz="0.0 0.0 ${-ur10_a2/2.0}" rpy="0 0 0" />
+          <mesh filename="package://ur_description/meshes/ur3/visual/upperarm.dae"/>
+        </geometry>
+        <material name="LightGrey">
+          <color rgba="0.7 0.7 0.7 1.0"/>
+        </material>
+      </visual>
+      <collision>
+        <geometry>
+          <mesh filename="package://ur_description/meshes/ur3/collision/upperarm.stl"/>
+        </geometry>
+      </collision>
+      <xacro:cylinder_inertial radius="0.075" length="${-ur3_a2}" mass="${upper_arm_mass}">
+        <origin xyz="0.0 0.0 ${-ur3_a2/2.0}" rpy="0 0 0" />
       </xacro:cylinder_inertial>
     </link>
@@ -150,17 +149,17 @@
       <visual>
          <geometry>
-          <mesh filename="package://ur_description/meshes/ur10/visual/forearm.dae"/>
-        </geometry>
-        <material name="LightGrey">
-          <color rgba="0.7 0.7 0.7 1.0"/>
-        </material>
-      </visual>
-      <collision>
-        <geometry>
-          <mesh filename="package://ur_description/meshes/ur10/collision/forearm.stl"/>
-        </geometry>
-      </collision>
-      <xacro:cylinder_inertial radius="0.075" length="${-ur10_a3}" mass="${forearm_mass}">
-        <origin xyz="0.0 0.0 ${-ur10_a3/2.0}" rpy="0 0 0" />
+          <mesh filename="package://ur_description/meshes/ur3/visual/forearm.dae"/>
+        </geometry>
+        <material name="LightGrey">
+          <color rgba="0.7 0.7 0.7 1.0"/>
+        </material>
+      </visual>
+      <collision>
+        <geometry>
+          <mesh filename="package://ur_description/meshes/ur3/collision/forearm.stl"/>
+        </geometry>
+      </collision>
+      <xacro:cylinder_inertial radius="0.075" length="${-ur3_a3}" mass="${forearm_mass}">
+        <origin xyz="0.0 0.0 ${-ur3_a3/2.0}" rpy="0 0 0" />
       </xacro:cylinder_inertial>
     </link>
@@ -181,13 +180,13 @@
       <visual>
         <geometry>
-          <mesh filename="package://ur_description/meshes/ur10/visual/wrist1.dae"/>
-        </geometry>
-        <material name="LightGrey">
-          <color rgba="0.7 0.7 0.7 1.0"/>
-        </material>
-      </visual>
-      <collision>
-        <geometry>
-          <mesh filename="package://ur_description/meshes/ur10/collision/wrist1.stl"/>
+          <mesh filename="package://ur_description/meshes/ur3/visual/wrist1.dae"/>
+        </geometry>
+        <material name="LightGrey">
+          <color rgba="0.7 0.7 0.7 1.0"/>
+        </material>
+      </visual>
+      <collision>
+        <geometry>
+          <mesh filename="package://ur_description/meshes/ur3/collision/wrist1.stl"/>
         </geometry>
       </collision>
@@ -212,13 +211,13 @@
       <visual>
         <geometry>
-          <mesh filename="package://ur_description/meshes/ur10/visual/wrist2.dae"/>
-        </geometry>
-        <material name="LightGrey">
-          <color rgba="0.7 0.7 0.7 1.0"/>
-        </material>
-      </visual>
-      <collision>
-        <geometry>
-          <mesh filename="package://ur_description/meshes/ur10/collision/wrist2.stl"/>
+          <mesh filename="package://ur_description/meshes/ur3/visual/wrist2.dae"/>
+        </geometry>
+        <material name="LightGrey">
+          <color rgba="0.7 0.7 0.7 1.0"/>
+        </material>
+      </visual>
+      <collision>
+        <geometry>
+          <mesh filename="package://ur_description/meshes/ur3/collision/wrist2.stl"/>
         </geometry>
       </collision>
@@ -243,13 +242,13 @@
       <visual>
         <geometry>
-          <mesh filename="package://ur_description/meshes/ur10/visual/wrist3.dae"/>
-        </geometry>
-        <material name="LightGrey">
-          <color rgba="0.7 0.7 0.7 1.0"/>
-        </material>
-      </visual>
-      <collision>
-        <geometry>
-          <mesh filename="package://ur_description/meshes/ur10/collision/wrist3.stl"/>
+          <mesh filename="package://ur_description/meshes/ur3/visual/wrist3.dae"/>
+        </geometry>
+        <material name="LightGrey">
+          <color rgba="0.7 0.7 0.7 1.0"/>
+        </material>
+      </visual>
+      <collision>
+        <geometry>
+          <mesh filename="package://ur_description/meshes/ur3/collision/wrist3.stl"/>
         </geometry>
       </collision>

File: urdf/ur3_joint_limited_robot.urdf.xacro (robot description, xacro)
@@ -1,11 +1,11 @@
 <?xml version="1.0"?>
 <robot xmlns:xacro="http://www.ros.org/wiki/xacro"
-       name="ur10" >
+       name="ur3" >
   <!-- common stuff -->
   <xacro:include filename="$(find ur_description)/urdf/common.gazebo.xacro" />
-  <!-- ur10 -->
-  <xacro:include filename="$(find ur_description)/urdf/ur10.urdf.xacro" />
+  <!-- ur3 -->
+  <xacro:include filename="$(find ur_description)/urdf/ur3.urdf.xacro" />
   <!-- arm -->
-  <xacro:ur10_robot prefix="" joint_limited="false"/>
+  <xacro:ur3_robot prefix="" joint_limited="true"/>
   <link name="world" />
   <joint name="world_joint" type="fixed">

File: urdf/ur3_robot.urdf.xacro (robot description, xacro)
@@ -1,11 +1,11 @@
 <?xml version="1.0"?>
 <robot xmlns:xacro="http://www.ros.org/wiki/xacro"
-       name="ur10" >
+       name="ur3" >
   <!-- common stuff -->
   <xacro:include filename="$(find ur_description)/urdf/common.gazebo.xacro" />
-  <!-- ur10 -->
-  <xacro:include filename="$(find ur_description)/urdf/ur10.urdf.xacro" />
+  <!-- ur3 -->
+  <xacro:include filename="$(find ur_description)/urdf/ur3.urdf.xacro" />
   <!-- arm -->
-  <xacro:ur10_robot prefix="" joint_limited="false"/>
+  <xacro:ur3_robot prefix="" joint_limited="false"/>
   <link name="world" />
   <joint name="world_joint" type="fixed">
